Commit message: Modèle plan 3D

File: urdf/env.urdf (robot description, URDF)
Before this commit: robot m2wr, 3 links, 2 joints
Links:
- removed link link_chassis
- removed link link_left_wheel
- removed link link_right_wheel
- added link table, mass 5; collision box size=0.5 0.3 0.07; visual box size=0.5 0.3 0.07
Joints:
- removed joint joint_left_wheel
- removed joint joint_right_wheel
